File: sch/power_backup_v2.sch (EAGLE design)
At the start: 38 parts, among them IC1 78L05SMD, IC2 ACS712-LC, K1 DS2Y-S-DC48V, T1 BC847, T2 BC847, T3 BC847, T4 BC847

Commit message: updated images
Parts:
- renumbered U$1 to K2
Other:
- moved on the sheet: D4, D5, R4, R5

Commit message: version 2
Parts:
- removed IC1: 78L05SMD, linear:78L05SMD
- removed K1: DS2Y-S-DC48V, relay:DS2Y-S-DC48V
- removed SV1: (no value), con-lstb:MA10-2
- added C5: (no value), rcl:CPOL-EUE3.5-8
- added D6: (no value), eagle-ltspice:DIODE_E-SMC
- added IC3: LM2576-ADJ, linear:LM2596S
- added JP1: (no value), pinhead:PINHD-1X4
- added L1: 220u, inductor-neosid:MS85
- added Q2: IRF3704S, transistor-power:IRF3704S
- added R13, R18: 1k, rcl:R-EU_M0805
- added R19: 6K2, rcl:R-EU_M0805
- added R20: 2K, rcl:R-EU_M0805
- added U$1: BALANCER, balancer20a:BALANCER
- added X1, X2: MSTBA5, con-phoenix-508:MSTBA5
- D3: value PMLL4150 -> (none); device diode:PMLL4150 -> diode:DIODE-DO214AA
- IC2: value ACS712-LC -> ACS712-5A
- LED1, LED2, LED3: device led:LED5MM -> led:LED3MM
- R12: value 560 -> 1k
Connections:
- removed net CON_VBATP: IC1G$1.VIN, K2G$2.MID, K2G$3.MID, R9.2, SV1.10, SV1.12
- removed net S_REL_IN: ARDUINO1.D13, R12.2
- removed net VOUT: IC2.IP-, IC2.IP-1, K2G$2.NO, K2G$3.NO
- new net BAT12V: IC3.IN, JP1.1, K2G$2.MID, K2G$3.MID, R9.2, U$1.12V
- new net BAT4V: JP1.3, U$1.4V
- new net BAT8V: JP1.2, U$1.8V
- new net N$16: R18.1, T4.B
- new net N$22: D3.C, IC3.OUT, L1.1
- new net N$23: IC3.FB, R19.2, R20.1
- new net N$4: C5.+, D6.C, Q2.D
- new net PWRP: IC2.IP-, IC2.IP-1, Q2.S
- new net S_PWR_REG: ARDUINO1.D10, R18.2
- net +5V: now also L1.2, R12.1, R19.1, X2-3.1; no longer IC1G$1.VOUT
- net CON_ERROR_OC: now also X2-5.1; no longer SV1.18, SV1.20
- net CON_PWR2P: now also D6.A, U$1.VIN; no longer K13.S, SV1.2, SV1.4
- net CON_PWRP: now also IC2.IP+, IC2.IP+1, X1-1.1; no longer D3.C, K11.+, K13.P, SV1.1, SV1.3
- net CON_RX: now also X1-5.1; no longer SV1.17, SV1.19
- net CON_TX: now also X1-4.1; no longer SV1.13, SV1.15
- net CON_VOUT: now also K2G$2.NO, K2G$3.NO, X2-1.1; no longer IC2.IP+, IC2.IP+1, SV1.11, SV1.9
- net GND: now also C5.-, D3.A, IC3.EN, IC3.GND, IC3.GND@1, JP1.4, R20.2, U$1.0V, U$1.GND, X1-2.1, X1-3.1, X2-2.1, X2-4.1; no longer IC1G$1.GND@1, IC1G$1.GND@2, IC1G$1.GND@3, IC1G$1.GND@4, SV1.14, SV1.16, SV1.5, SV1.6, SV1.7, SV1.8
- net N$10: now also R12.2, R13.2, T4.C; no longer R12.1, T4.B
- net N$11: now also Q2.G, R13.1; no longer D3.A, K11.-, T4.C
Other:
- moved on the sheet: C3, C4, D3, R12, R4, T4
